Commit message: edit launch files for cob3_defs

File: cob3_simulation/cob3_defs/ros/defs/LaserBlock.urdf (robot description, URDF)
Before this commit: robot LaserBlock, 1 links, 1 joints
Links:
- removed link laser_block
- added link base_laser_front, mass 1.0; collision box size=0.1 0.1 0.1; visual box size=0.1 0.1 0.1
Joints:
- joint base_world_joint: child laser_block -> base_laser_front
