Commit message: changes to urdf models

File: cob3_simulation/cob3_defs/ros/defs/platform.urdf (robot description, URDF)
Before this commit: robot torso, 9 links, 8 joints
Links:
- link link_platform: geometry collision mesh filename=package://cob3_defs/common/files/meshes/platform.stl; visual mesh filename=package://cob3_defs/common/files/meshes/platform.stl

File: cob3_simulation/cob3_defs/ros/defs/torso.urdf (robot description, URDF)
Before this commit: robot torso, 10 links, 9 joints
Links:
- removed link link_torso
- added link link_platform, mass 80; collision mesh filename=package://cob3_defs/common/files/meshes/platform.stl; visual mesh filename=package://cob3_defs/common/files/meshes/platform.stl
- added link link_steerFL, mass 1; collision box size=0.001 0.001 0.001; visual box size=0.001 0.001 0.001
- added link link_steerFR, mass 1; collision box size=0.001 0.001 0.001; visual box size=0.001 0.001 0.001
- added link link_steerRL, mass 1; collision box size=0.001 0.001 0.001; visual box size=0.001 0.001 0.001
- added link link_steerRR, mass 1; collision box size=0.001 0.001 0.001; visual box size=0.001 0.001 0.001
- added link link_wheelFL, mass 1; collision cylinder length=0.05 radius=0.1; visual cylinder length=0.05 radius=0.1
- added link link_wheelFR, mass 1; collision cylinder length=0.05 radius=0.1; visual cylinder length=0.05 radius=0.1
- added link link_wheelRL, mass 1; collision cylinder length=0.05 radius=0.1; visual cylinder length=0.05 radius=0.1
- added link link_wheelRR, mass 1; collision cylinder length=0.05 radius=0.1; visual cylinder length=0.05 radius=0.1
- link link_colorcameraLeft: mass 0.1 -> 1; geometry collision box size=0.01 0.01 0.01; visual box size=0.01 0.01 0.01
- link link_colorcameraRight: mass 0.1 -> 1; geometry collision box size=0.01 0.01 0.01; visual box size=0.01 0.01 0.01
- link link_eyes: mass 0.1 -> 1
- link link_head: mass 0.1 -> 1; geometry collision mesh filename=package://cob3_defs/common/files/meshes/head.stl; visual mesh filename=package://cob3_defs/common/files/meshes/head.stl
- link link_headZ: mass 0.001 -> 0.1
- link link_neck: mass 0.1 -> 1; geometry collision mesh filename=package://cob3_defs/common/files/meshes/neck.stl; visual mesh filename=package://cob3_defs/common/files/meshes/neck.stl
- link link_neckZ: mass 0.001 -> 0.1
- link link_swissranger: mass 0.1 -> 1; geometry collision box size=0.01 0.01 0.01; visual box size=0.01 0.01 0.01
Joints:
- removed joint joint_torso_neckZ
- removed joint joint_torso_tray
- added joint joint_platform_neckZ: type revolute, parent link_platform, child link_neckZ, origin xyz=0.24627 0 0.7798 rpy=0 0 0, axis 0 0 1, limit lower=-0.5 upper=0.5 effort=100 velocity=1.0
- added joint joint_platform_steerFL: type continuous, parent link_platform, child link_steerFL, origin xyz=0.235 0.1825 0.092 rpy=0 0 0, axis 0 0 1, limit lower=-1 upper=1 effort=100 velocity=5
- added joint joint_platform_steerFR: type continuous, parent link_platform, child link_steerFR, origin xyz=0.235 -0.1825 0.092 rpy=0 0 0, axis 0 0 1, limit lower=-1 upper=1 effort=100 velocity=5
- added joint joint_platform_steerRL: type continuous, parent link_platform, child link_steerRL, origin xyz=-0.235 0.1825 0.092 rpy=0 0 0, axis 0 0 1, limit lower=-1 upper=1 effort=100 velocity=5
- added joint joint_platform_steerRR: type continuous, parent link_platform, child link_steerRR, origin xyz=-0.235 -0.1825 0.092 rpy=0 0 0, axis 0 0 1, limit lower=-1 upper=1 effort=100 velocity=5
- added joint joint_platform_tray: type revolute, parent link_platform, child link_tray, origin xyz=0.5 0 0.8 rpy=0 0 0, axis 0 0 1, limit lower=-1 upper=1 effort=100 velocity=5
- added joint joint_steerFL_wheelFL: type continuous, parent link_steerFL, child link_wheelFL, origin xyz=0 0 0.001 rpy=0 0 0, axis 0 1 0, limit lower=-1 upper=1 effort=100 velocity=5
- added joint joint_steerFR_wheelFR: type continuous, parent link_steerFR, child link_wheelFR, origin xyz=0 0 0.001 rpy=0 0 0, axis 0 1 0, limit lower=-1 upper=1 effort=100 velocity=5
- added joint joint_steerRL_wheelRL: type continuous, parent link_steerRL, child link_wheelRL, origin xyz=0 0 0.001 rpy=0 0 0, axis 0 1 0, limit lower=-1 upper=1 effort=100 velocity=5
- added joint joint_steerRR_wheelRR: type continuous, parent link_steerRR, child link_wheelRR, origin xyz=0 0 0.001 rpy=0 0 0, axis 0 1 0, limit lower=-1 upper=1 effort=100 velocity=5
- joint joint_eyes_colorcameraLeft: origin xyz=0.05 0.1 0 rpy=0 0 0 -> xyz=0.075 0.05 0 rpy=0 0 0
- joint joint_eyes_colorcameraRight: origin xyz=0.05 -0.1 0 rpy=0 0 0 -> xyz=0.075 -0.05 0 rpy=0 0 0
- joint joint_eyes_swissranger: origin xyz=0.05 0 0 rpy=0 0 0 -> xyz=0.075 0 0 rpy=0 0 0
- joint joint_headZ_head: origin xyz=0 0 0 rpy=0 0 0 -> xyz=0 0 0.001 rpy=0 0 0
- joint joint_head_eyes: origin xyz=0 0 0.1 rpy=0 0 0 -> xyz=-0.1 0 0.2 rpy=0 0 0
- joint joint_neckZ_neck: limit lower=-1 upper=1 effort=100 velocity=5 -> lower=-0.5 upper=0.5 effort=100 velocity=1.0; origin xyz=0 0 0 rpy=0 0 0 -> xyz=0 0 0.001 rpy=0 0 0
- joint joint_neck_headZ: origin xyz=0 0 0.1 rpy=0 0 0 -> xyz=-0.09039 0 0.30489 rpy=0 0 0

File: cob3_simulation/cob3_defs/ros/robots/cob3.urdf.xacro (robot description, xacro)
@@ -6,19 +6,19 @@
 	<!-- include gazebo defs-->
 	<include filename="$(find cob3_defs)/ros/defs/gazebo.urdf" />
-	<!-- include platform defs-->
-	<include filename="$(find cob3_defs)/ros/defs/platform.urdf" />
+	<!-- create joint to world -->
+	<joint name="joint_world_platform" type="fixed">
+		<origin xyz="0 0 0" rpy="0 0 0" />
+		<parent link="world"/>
+		<child link="link_platform"/>
+	</joint>
 	<!-- include torso defs-->
 	<include filename="$(find cob3_defs)/ros/defs/torso.urdf" />
+	<!-- include sensor defs-->
 	<include filename="$(find cob3_defs)/ros/defs/torso_sensors.urdf" />
-	<joint name="joint_basePlate_torso" type="fixed">
-		<origin xyz="0 0 0.5" rpy="0 0 0" />
-		<parent link="link_platform"/>
-		<child link="link_torso"/>
-	</joint>
 	<!-- include arm defs-->
 	<include filename="$(find cob3_defs)/ros/defs/arm.urdf" />
-	<joint name="joint_torso_arm0" type="fixed">
-		<origin xyz="-0.1 0 0.3" rpy="0.5 0 0" />
-		<parent link="link_torso"/>
+	<joint name="joint_platform_arm0" type="fixed">
+		<origin xyz="0 0 0.8" rpy="0.5 0 0" /> <!-- TODO: put in real transformation from platform to arm0-->
+		<parent link="link_platform"/>
 		<child link="link_arm0"/>
 	</joint>

File: cob3_simulation/cob3_defs/ros/robots/cob3_torso.urdf.xacro (robot description, xacro)
@@ -7,8 +7,8 @@
 	<include filename="$(find cob3_defs)/ros/defs/gazebo.urdf" />
 	<!-- create joint to world -->
-	<joint name="joint_world_torso" type="fixed">
+	<joint name="joint_world_platform" type="fixed">
 		<origin xyz="0 0 0" rpy="0 0 0" />
 		<parent link="world"/>
-		<child link="link_torso"/>
+		<child link="link_platform"/>
 	</joint>
 	<!-- include torso defs-->
