Commit message: added actor to joint

File: cob3_simulation/cob3_defs/ros/defs/sdh.urdf (robot description, URDF)
Before this commit: robot SDH, 10 links, 10 joints
Links:
- link Thumb-3: mass 1 -> 10
Joints:
- joint Thumb-2_Thumb-3: limit lower=-6.283185306 upper=6.283185306 effort=30 velocity=1.0 -> lower=-1 upper=1 effort=100 velocity=5

Commit message: adjust transformations and added motors to sdh gazebo model

File: cob3_simulation/cob3_defs/ros/defs/sdh.urdf (robot description, URDF)
Before this commit: robot SDH, 10 links, 10 joints
Links:
- removed link Finger1-1
- removed link Finger1-2
- removed link Finger1-3
- removed link Finger2-1
- removed link Finger2-2
- removed link Finger2-3
- removed link Palm
- removed link Thumb-1
- removed link Thumb-2
- removed link Thumb-3
- added link link_finger1-1, mass 0.1; collision mesh filename=package://cob3_defs/common/files/meshes/knuckle.stl; visual mesh filename=package://cob3_defs/common/files/meshes/knuckle.stl
- added link link_finger1-2, mass 0.1; collision mesh filename=package://cob3_defs/common/files/meshes/finger.stl; visual mesh filename=package://cob3_defs/common/files/meshes/finger.stl
- added link link_finger1-3, mass 0.1; collision mesh filename=package://cob3_defs/common/files/meshes/finger_tip.stl; visual mesh filename=package://cob3_defs/common/files/meshes/finger_tip.stl
- added link link_finger2-1, mass 0.1; collision mesh filename=package://cob3_defs/common/files/meshes/knuckle.stl; visual mesh filename=package://cob3_defs/common/files/meshes/knuckle.stl
- added link link_finger2-2, mass 0.1; collision mesh filename=package://cob3_defs/common/files/meshes/finger.stl; visual mesh filename=package://cob3_defs/common/files/meshes/finger.stl
- added link link_finger2-3, mass 0.1; collision mesh filename=package://cob3_defs/common/files/meshes/finger_tip.stl; visual mesh filename=package://cob3_defs/common/files/meshes/finger_tip.stl
- added link link_palm, mass 1; collision mesh filename=package://cob3_defs/common/files/meshes/palm.stl; visual mesh filename=package://cob3_defs/common/files/meshes/palm.stl
- added link link_thumb1, mass 0.1; collision mesh filename=package://pr2_defs/meshes/knuckle.stl; visual mesh filename=package://cob3_defs/common/files/meshes/knuckle.stl
- added link link_thumb2, mass 0.1; collision mesh filename=package://pr2_defs/meshes/finger.stl; visual mesh filename=package://cob3_defs/common/files/meshes/finger.stl
- added link link_thumb3, mass 0.1; collision mesh filename=package://cob3_defs/common/files/meshes/finger_tip.stl; visual mesh filename=package://cob3_defs/common/files/meshes/finger_tip.stl
Joints:
- removed joint Thumb-1_Thumb-2
- removed joint Thumb-2_Thumb-3
- removed joint World_palm
- removed joint finger1-1_finger1-2
- removed joint finger1-2_finger1-3
- removed joint finger2-1_finger2-2
- removed joint finger2-2_finger2-3
- removed joint palm_Thumb-1
- removed joint palm_finger1-1
- removed joint palm_finger2-1
- added joint joint_finger1-1_finger1-2: type revolute, parent link_finger1-1, child link_finger1-2, origin xyz=0 0 0.0165 rpy=0 0 0, axis 0 1 0, limit lower=-0.5 upper=0.5 effort=30 velocity=1.0
- added joint joint_finger1-2_finger1-3: type revolute, parent link_finger1-2, child link_finger1-3, origin xyz=0 0 0.0865 rpy=0 0 0, axis 0 1 0, limit lower=-0.5 upper=0.5 effort=30 velocity=1.0
- added joint joint_finger2-1_finger2-2: type revolute, parent link_finger2-1, child link_finger2-2, origin xyz=0 0 0.0165 rpy=0 0 0, axis 0 1 0, limit lower=-0.5 upper=0.5 effort=30 velocity=1.0
- added joint joint_finger2-2_finger2-3: type revolute, parent link_finger2-2, child link_finger2-3, origin xyz=0 0 0.0865 rpy=0 0 0, axis 0 1 0, limit lower=-0.5 upper=0.5 effort=30 velocity=1.0
- added joint joint_palm_finger1-1: type revolute, parent link_palm, child link_finger1-1, origin xyz=0.01905 0.033 0.0745 rpy=0 0 3.159265, axis 0 0 1, limit lower=-0.5 upper=0.5 effort=30 velocity=1.0
- added joint joint_palm_finger2-1: type revolute, parent link_palm, child link_finger2-1, origin xyz=0.01905 -0.033 0.0745 rpy=0 0 3.14159265, axis 0 0 1, limit lower=-0.5 upper=0.5 effort=30 velocity=1.0
- added joint joint_palm_thumb1: type revolute, parent link_palm, child link_thumb1, origin xyz=-0.03811 0 0.0745  rpy=0 0 0, axis 0 0 1, limit lower=-1 upper=1 effort=100 velocity=5
- added joint joint_thumb1_thumb2: type revolute, parent link_thumb1, child link_thumb2, origin xyz=0 0 0.0165 rpy=0 0 0, axis 0 1 0, limit lower=-1 upper=1 effort=100 velocity=5
- added joint joint_thumb2_thumb3: type revolute, parent link_thumb2, child link_thumb3, origin xyz=0 0 0.0865 rpy=0 0 0, axis 0 1 0, limit lower=-1 upper=1 effort=100 velocity=5
- added joint joint_world_palm: type fixed, parent world, child link_palm, origin xyz=0 0 0 rpy=0 0 0

Commit message: changes in file structure

File: cob3_simulation/cob3_defs/ros/defs/sdh.urdf (robot description, URDF)
Before this commit: robot sdh, 10 links, 10 joints
Joints:
- removed joint joint_world_palm
- added joint joint_armTCP_palm: type fixed, parent link_arm7, child link_palm, origin xyz=0 0 0.1125 rpy=0 0 0

Commit message: adjust armTCP offset

File: cob3_simulation/cob3_defs/ros/defs/sdh.urdf (robot description, URDF)
Before this commit: robot sdh, 10 links, 10 joints
Joints:
- joint joint_armTCP_palm: origin xyz=0 0 0.1125 rpy=0 0 0 -> xyz=0 0 0.1126 rpy=0 0 0

Commit message: changed directory to cob3_defs

File: cob3_simulation/cob3_defs/ros/defs/sdh.urdf (robot description, URDF)
Before this commit: robot sdh, 10 links, 9 joints
Links:
- link link_thumb1: geometry collision mesh filename=package://cob3_defs/common/files/meshes/knuckle.stl; visual mesh filename=package://cob3_defs/common/files/meshes/knuckle.stl
- link link_thumb2: geometry collision mesh filename=package://cob3_defs/common/files/meshes/finger.stl; visual mesh filename=package://cob3_defs/common/files/meshes/finger.stl

Commit message: changed sdh finger names

File: cob3_simulation/cob3_defs/ros/defs/sdh.urdf (robot description, URDF)
Before this commit: robot sdh, 10 links, 9 joints
Links:
- removed link link_finger1-1
- removed link link_finger1-2
- removed link link_finger1-3
- removed link link_finger2-1
- removed link link_finger2-2
- removed link link_finger2-3
- added link link_finger11, mass 0.1; collision mesh filename=package://cob3_defs/common/files/meshes/knuckle.stl; visual mesh filename=package://cob3_defs/common/files/meshes/knuckle.stl
- added link link_finger12, mass 0.1; collision mesh filename=package://cob3_defs/common/files/meshes/finger.stl; visual mesh filename=package://cob3_defs/common/files/meshes/finger.stl
- added link link_finger13, mass 0.1; collision mesh filename=package://cob3_defs/common/files/meshes/finger_tip.stl; visual mesh filename=package://cob3_defs/common/files/meshes/finger_tip.stl
- added link link_finger21, mass 0.1; collision mesh filename=package://cob3_defs/common/files/meshes/knuckle.stl; visual mesh filename=package://cob3_defs/common/files/meshes/knuckle.stl
- added link link_finger22, mass 0.1; collision mesh filename=package://cob3_defs/common/files/meshes/finger.stl; visual mesh filename=package://cob3_defs/common/files/meshes/finger.stl
- added link link_finger23, mass 0.1; collision mesh filename=package://cob3_defs/common/files/meshes/finger_tip.stl; visual mesh filename=package://cob3_defs/common/files/meshes/finger_tip.stl
Joints:
- removed joint joint_finger1-1_finger1-2
- removed joint joint_finger1-2_finger1-3
- removed joint joint_finger2-1_finger2-2
- removed joint joint_finger2-2_finger2-3
- removed joint joint_palm_finger1-1
- removed joint joint_palm_finger2-1
- added joint joint_finger11_finger12: type revolute, parent link_finger11, child link_finger12, origin xyz=0 0 0.0165 rpy=0 0 0, axis 0 1 0, limit lower=-0.5 upper=0.5 effort=100 velocity=1.0
- added joint joint_finger12_finger13: type revolute, parent link_finger12, child link_finger13, origin xyz=0 0 0.0865 rpy=0 0 0, axis 0 1 0, limit lower=-0.5 upper=0.5 effort=100 velocity=1.0
- added joint joint_finger21_finger22: type revolute, parent link_finger21, child link_finger22, origin xyz=0 0 0.0165 rpy=0 0 0, axis 0 1 0, limit lower=-0.5 upper=0.5 effort=100 velocity=1.0
- added joint joint_finger22_finger23: type revolute, parent link_finger22, child link_finger23, origin xyz=0 0 0.0865 rpy=0 0 0, axis 0 1 0, limit lower=-0.5 upper=0.5 effort=100 velocity=1.0
- added joint joint_palm_finger11: type revolute, parent link_palm, child link_finger11, origin xyz=0.01905 0.033 0.0745 rpy=0 0 3.159265, axis 0 0 1, limit lower=-0.5 upper=0.5 effort=100 velocity=1.0
- added joint joint_palm_finger21: type revolute, parent link_palm, child link_finger21, origin xyz=0.01905 -0.033 0.0745 rpy=0 0 3.14159265, axis 0 0 1, limit lower=-0.5 upper=0.5 effort=100 velocity=1.0

Commit message: update sdh urdf

File: cob3_simulation/cob3_defs/ros/defs/sdh.urdf (robot description, URDF)
Before this commit: robot sdh, 10 links, 9 joints
Joints:
- joint joint_finger11_finger12: limit lower=-0.5 upper=0.5 effort=100 velocity=1.0 -> lower=-2 upper=2 effort=100 velocity=5
- joint joint_finger12_finger13: limit lower=-0.5 upper=0.5 effort=100 velocity=1.0 -> lower=-2 upper=2 effort=100 velocity=5
- joint joint_finger21_finger22: limit lower=-0.5 upper=0.5 effort=100 velocity=1.0 -> lower=-2 upper=2 effort=100 velocity=5
- joint joint_finger22_finger23: limit lower=-0.5 upper=0.5 effort=100 velocity=1.0 -> lower=-2 upper=2 effort=100 velocity=5
- joint joint_palm_finger11: limit lower=-0.5 upper=0.5 effort=100 velocity=1.0 -> lower=-2 upper=2 effort=100 velocity=5
- joint joint_palm_finger21: limit lower=-0.5 upper=0.5 effort=100 velocity=1.0 -> lower=-2 upper=2 effort=100 velocity=5
- joint joint_palm_thumb1: limit lower=-1 upper=1 effort=100 velocity=5 -> lower=-2 upper=2 effort=100 velocity=5
- joint joint_thumb1_thumb2: limit lower=-1 upper=1 effort=100 velocity=5 -> lower=-2 upper=2 effort=100 velocity=5
- joint joint_thumb2_thumb3: limit lower=-1 upper=1 effort=100 velocity=5 -> lower=-2 upper=2 effort=100 velocity=5
