Commit message: added urdf description of arm

File: cob3_simulation/cob3_defs/ros/defs/arm.urdf (robot description, URDF)
Before this commit: robot SchunkArmLWA3, 7 links, 7 joints
Links:
- removed link Arm1
- removed link Arm2
- removed link Arm3
- removed link Arm4
- removed link Arm5
- removed link Arm6
- removed link End
- added link link_arm0, mass 2; collision cylinder length=0.01 radius=0.1; visual cylinder length=0.01 radius=0.1
- added link link_arm1, mass 2; collision mesh filename=package://cob3_defs/common/files/meshes/arm1.stl; visual mesh filename=package://cob3_defs/common/files/meshes/arm1.stl
- added link link_arm2, mass 2; collision mesh filename=package://cob3_defs/common/files/meshes/arm2.stl; visual mesh filename=package://cob3_defs/common/files/meshes/arm2.stl
- added link link_arm3, mass 2; collision mesh filename=package://cob3_defs/common/files/meshes/arm3.stl; visual mesh filename=package://cob3_defs/common/files/meshes/arm3.stl
- added link link_arm4, mass 2; collision mesh filename=package://cob3_defs/common/files/meshes/arm4.stl; visual mesh filename=package://cob3_defs/common/files/meshes/arm4.stl
- added link link_arm5, mass 2; collision mesh filename=package://cob3_defs/common/files/meshes/arm5.stl; visual mesh filename=package://cob3_defs/common/files/meshes/arm5.stl
- added link link_arm6, mass 2; collision mesh filename=package://cob3_defs/common/files/meshes/arm6.stl; visual mesh filename=package://cob3_defs/common/files/meshes/arm6.stl
- added link link_arm7, mass 2; collision mesh filename=package://cob3_defs/common/files/meshes/arm7.stl; visual mesh filename=package://cob3_defs/common/files/meshes/arm7.stl
Joints:
- removed joint par_World_joint1
- removed joint par_joint2_joint3
- removed joint par_joint4_joint5
- removed joint par_joint6_End
- removed joint per_joint1_joint2
- removed joint per_joint3_joint4
- removed joint per_joint5_joint6
- added joint joint_arm0_arm1: type revolute, parent link_arm0, child link_arm1, origin xyz=0 0 0.01 rpy=0 0 0, axis 0 0 1, limit lower=-0.5 upper=0.5 effort=100 velocity=0.01
- added joint joint_arm1_arm2: type revolute, parent link_arm1, child link_arm2, origin xyz=0 0 0.25 rpy=0 0 0, axis 0 1 0, limit lower=-0.5 upper=0.5 effort=100 velocity=0.01
- added joint joint_arm2_arm3: type revolute, parent link_arm2, child link_arm3, origin xyz=0 0 0.110 rpy=0 0 0, axis 0 0 1, limit lower=-0.5 upper=0.5 effort=100 velocity=0.01
- added joint joint_arm3_arm4: type revolute, parent link_arm3, child link_arm4, origin xyz=0 0 0.298 rpy=0 0 0, axis 0 1 0, limit lower=-0.5 upper=0.5 effort=100 velocity=0.01
- added joint joint_arm4_arm5: type revolute, parent link_arm4, child link_arm5, origin xyz=0 0 0.100 rpy=0 0 0, axis 0 0 1, limit lower=-0.5 upper=0.5 effort=100 velocity=0.01
- added joint joint_arm5_arm6: type revolute, parent link_arm5, child link_arm6, origin xyz=0 0 0.2165 rpy=0 0 0, axis 0 1 0, limit lower=-0.5 upper=0.5 effort=100 velocity=0.01
- added joint joint_arm6_arm7: type revolute, parent link_arm6, child link_arm7, origin xyz=0 0 0.080 rpy=0 0 0, axis 0 0 1, limit lower=-0.5 upper=0.5 effort=100 velocity=0.01
- added joint joint_world_arm0: type fixed, parent world, child link_arm0, origin xyz=0 0 0 rpy=0 0 0

File: cob3_simulation/cob3_defs/ros/defs/sdh.urdf (robot description, URDF)
Before this commit: robot SDH, 10 links, 10 joints
Joints:
- joint joint_finger1-1_finger1-2: limit lower=-0.5 upper=0.5 effort=30 velocity=1.0 -> lower=-0.5 upper=0.5 effort=100 velocity=1.0
- joint joint_finger1-2_finger1-3: limit lower=-0.5 upper=0.5 effort=30 velocity=1.0 -> lower=-0.5 upper=0.5 effort=100 velocity=1.0
- joint joint_finger2-1_finger2-2: limit lower=-0.5 upper=0.5 effort=30 velocity=1.0 -> lower=-0.5 upper=0.5 effort=100 velocity=1.0
- joint joint_finger2-2_finger2-3: limit lower=-0.5 upper=0.5 effort=30 velocity=1.0 -> lower=-0.5 upper=0.5 effort=100 velocity=1.0
- joint joint_palm_finger1-1: limit lower=-0.5 upper=0.5 effort=30 velocity=1.0 -> lower=-0.5 upper=0.5 effort=100 velocity=1.0
- joint joint_palm_finger2-1: limit lower=-0.5 upper=0.5 effort=30 velocity=1.0 -> lower=-0.5 upper=0.5 effort=100 velocity=1.0

Commit message: added torso and transformation changes

File: cob3_simulation/cob3_defs/ros/defs/arm.urdf (robot description, URDF)
Before this commit: robot arm, 8 links, 8 joints
Links:
- link link_arm0: geometry collision box size=0.1 0.1 0.1; visual box size=0.1 0.1 0.1
Joints:
- removed joint joint_world_arm0
- joint joint_arm0_arm1: origin xyz=0 0 0.01 rpy=0 0 0 -> xyz=0 0 0.1 rpy=0 0 0

File: cob3_simulation/cob3_defs/ros/defs/sdh.urdf (robot description, URDF)
Before this commit: robot sdh, 10 links, 10 joints
Joints:
- removed joint joint_armTCP_palm

File: cob3_simulation/cob3_defs/ros/robots/cob3.urdf.xacro (robot description, xacro)
@@ -6,7 +6,30 @@
 	<!-- include gazebo defs-->
 	<include filename="$(find cob3_defs)/ros/defs/gazebo.urdf" />
+	<!-- create joint to world -->
+	<joint name="joint_world_torso" type="fixed">
+		<origin xyz="0 0 0" rpy="0 0 0" />
+		<parent link="world"/>
+		<child link="link_torso"/>
+	</joint>
+	<!-- include torso defs-->
+	<include filename="$(find cob3_defs)/ros/defs/torso.urdf" />
+	<joint name="joint_basePlate_torso" type="fixed">
+		<origin xyz="0 0 0.1126" rpy="0 0 0" />
+		<parent link="link_base_Plate"/>
+		<child link="link_torso"/>
+	</joint>
 	<!-- include arm defs-->
 	<include filename="$(find cob3_defs)/ros/defs/arm.urdf" />
+	<joint name="joint_torso_arm0" type="fixed">
+		<origin xyz="-0.1 0 0.3" rpy="0.5 0 0" />
+		<parent link="link_torso"/>
+		<child link="link_arm0"/>
+	</joint>
 	<!-- include sdh defs-->
 	<include filename="$(find cob3_defs)/ros/defs/sdh.urdf" />
+  	<joint name="joint_arm7_palm" type="fixed">
+		<origin xyz="0 0 0.1126" rpy="0 0 0" />
+		<parent link="link_arm7"/>
+		<child link="link_palm"/>
+	</joint>
 </robot>

File: cob3_simulation/cob3_defs/ros/robots/cob3_arm.urdf.xacro (robot description, xacro)
@@ -6,4 +6,10 @@
 	<!-- include gazebo defs-->
 	<include filename="$(find cob3_defs)/ros/defs/gazebo.urdf" />
+	<!-- create joint to world -->
+	<joint name="joint_world_arm0" type="fixed">
+		<origin xyz="0 0 0" rpy="0 0 0" />
+		<parent link="world"/>
+		<child link="link_arm0"/>
+	</joint>
 	<!-- include arm defs-->
 	<include filename="$(find cob3_defs)/ros/defs/arm.urdf" />

File: cob3_simulation/cob3_defs/ros/robots/cob3_torso.urdf.xacro (robot description, xacro)
@@ -1,4 +1,4 @@
 <?xml version="1.0"?>
-<robot name="cob3_sdh"
+<robot name="cob3_torso"
 	xmlns:sensor="http://playerstage.sourceforge.net/gazebo/xmlschema/#sensor"
 	xmlns:controller="http://playerstage.sourceforge.net/gazebo/xmlschema/#controller"
@@ -7,10 +7,10 @@
 	<include filename="$(find cob3_defs)/ros/defs/gazebo.urdf" />
 	<!-- create joint to world -->
-	<joint name="joint_world_palm" type="fixed">
+	<joint name="joint_world_torso" type="fixed">
 		<origin xyz="0 0 0" rpy="0 0 0" />
 		<parent link="world"/>
-		<child link="link_palm"/>
+		<child link="link_torso"/>
 	</joint>
-	<!-- include sdh defs-->
-	<include filename="$(find cob3_defs)/ros/defs/sdh.urdf" />
+	<!-- include torso defs-->
+	<include filename="$(find cob3_defs)/ros/defs/torso.urdf" />
 </robot>

Commit message: new stl files for arm0 and arm1; added camera sensors to torso

File: cob3_simulation/cob3_defs/ros/defs/arm.urdf (robot description, URDF)
Before this commit: robot arm, 8 links, 7 joints
Links:
- link link_arm0: mass 2 -> 1; geometry collision mesh filename=package://cob3_defs/common/files/meshes/arm0.stl; visual mesh filename=package://cob3_defs/common/files/meshes/arm0.stl
Joints:
- joint joint_arm0_arm1: origin xyz=0 0 0.1 rpy=0 0 0 -> xyz=0 0 0.0569 rpy=0 0 0
- joint joint_arm1_arm2: origin xyz=0 0 0.25 rpy=0 0 0 -> xyz=0 0 0.1931 rpy=0 0 0

File: cob3_simulation/cob3_defs/ros/defs/torso.urdf (robot description, URDF)
Before this commit: robot torso, 10 links, 9 joints
Links:
- link link_torso: mass 0.1 -> 20
- link link_tray: mass 0.1 -> 5

File: cob3_simulation/cob3_defs/ros/robots/cob3.urdf.xacro (robot description, xacro)
@@ -6,8 +6,9 @@
 	<!-- include gazebo defs-->
 	<include filename="$(find cob3_defs)/ros/defs/gazebo.urdf" />
-	<!-- include torso defs-->
+	<!-- include platform defs-->
 	<include filename="$(find cob3_defs)/ros/defs/platform.urdf" />
 	<!-- include torso defs-->
 	<include filename="$(find cob3_defs)/ros/defs/torso.urdf" />
+	<include filename="$(find cob3_defs)/ros/defs/torso_sensors.urdf" />
 	<joint name="joint_basePlate_torso" type="fixed">
 		<origin xyz="0 0 0.5" rpy="0 0 0" />

File: cob3_simulation/cob3_defs/ros/robots/cob3_torso.urdf.xacro (robot description, xacro)
@@ -14,3 +14,5 @@
 	<!-- include torso defs-->
 	<include filename="$(find cob3_defs)/ros/defs/torso.urdf" />
+	<!-- include sensor defs-->
+	<include filename="$(find cob3_defs)/ros/defs/torso_sensors.urdf" />
 </robot>

Commit message: update of arm urdf

File: cob3_simulation/cob3_defs/ros/defs/arm.urdf (robot description, URDF)
Before this commit: robot arm, 8 links, 7 joints
Joints:
- joint joint_arm0_arm1: limit lower=-0.5 upper=0.5 effort=100 velocity=0.01 -> lower=-6.2831853 upper=6.2831853 effort=100 velocity=0.01
- joint joint_arm1_arm2: limit lower=-0.5 upper=0.5 effort=100 velocity=0.01 -> lower=-2.0943951 upper=2.0943951 effort=100 velocity=0.01
- joint joint_arm2_arm3: limit lower=-0.5 upper=0.5 effort=100 velocity=0.01 -> lower=-6.2831853 upper=6.2831853 effort=100 velocity=0.01
- joint joint_arm3_arm4: limit lower=-0.5 upper=0.5 effort=100 velocity=0.01 -> lower=-2.0943951 upper=2.0943951 effort=100 velocity=0.01
- joint joint_arm4_arm5: limit lower=-0.5 upper=0.5 effort=100 velocity=0.01 -> lower=-6.2831853 upper=6.2831853 effort=100 velocity=0.01
- joint joint_arm5_arm6: limit lower=-0.5 upper=0.5 effort=100 velocity=0.01 -> lower=-2.0943951 upper=2.0943951 effort=100 velocity=0.01
- joint joint_arm6_arm7: limit lower=-0.5 upper=0.5 effort=100 velocity=0.01 -> lower=-6.2831853 upper=6.2831853 effort=100 velocity=0.01

Commit message: new package cob3_arm_ik

File: cob3_simulation/cob3_defs/ros/defs/arm.urdf (robot description, URDF)
Before this commit: robot arm, 8 links, 7 joints
Links:
- link link_arm2: mass 2 -> 0.2
- link link_arm3: mass 2 -> 0.2
- link link_arm4: mass 2 -> 0.2
- link link_arm5: mass 2 -> 0.2
- link link_arm6: mass 2 -> 0.2
- link link_arm7: mass 2 -> 0.2
Joints:
- joint joint_arm0_arm1: limit lower=-6.2831853 upper=6.2831853 effort=100 velocity=0.01 -> lower=-6.2831853 upper=6.2831853 effort=320 velocity=2.0
- joint joint_arm1_arm2: limit lower=-2.0943951 upper=2.0943951 effort=100 velocity=0.01 -> lower=-2.0943951 upper=2.0943951 effort=320 velocity=2.0
- joint joint_arm2_arm3: limit lower=-6.2831853 upper=6.2831853 effort=100 velocity=0.01 -> lower=-6.2831853 upper=6.2831853 effort=320 velocity=2.0
- joint joint_arm3_arm4: limit lower=-2.0943951 upper=2.0943951 effort=100 velocity=0.01 -> lower=-2.0943951 upper=2.0943951 effort=320 velocity=2.0
- joint joint_arm4_arm5: limit lower=-6.2831853 upper=6.2831853 effort=100 velocity=0.01 -> lower=-6.2831853 upper=6.2831853 effort=320 velocity=2.0
- joint joint_arm5_arm6: limit lower=-2.0943951 upper=2.0943951 effort=100 velocity=0.01 -> lower=-2.0943951 upper=2.0943951 effort=320 velocity=2.0
- joint joint_arm6_arm7: limit lower=-6.2831853 upper=6.2831853 effort=100 velocity=0.01 -> lower=-6.2831853 upper=6.2831853 effort=320 velocity=2.0

Commit message: adujst arm defs to real powercube values and changed from singleJointController to JointTrajectoryController

File: cob3_simulation/cob3_defs/ros/defs/arm.urdf (robot description, URDF)
Before this commit: robot arm, 8 links, 7 joints
Links:
- link link_arm0: mass 1 -> 1.8
- link link_arm1: mass 2 -> 3.6
- link link_arm2: mass 0.2 -> 2.8
- link link_arm3: mass 0.2 -> 2.0
- link link_arm4: mass 0.2 -> 1.6
- link link_arm5: mass 0.2 -> 1.2
- link link_arm6: mass 0.2 -> 1.1
- link link_arm7: mass 0.2 -> 0.5
Joints:
- removed joint joint_arm0_arm1
- removed joint joint_arm1_arm2
- removed joint joint_arm2_arm3
- removed joint joint_arm3_arm4
- removed joint joint_arm4_arm5
- removed joint joint_arm5_arm6
- removed joint joint_arm6_arm7
- added joint joint_arm1: type revolute, parent link_arm0, child link_arm1, origin xyz=0 0 0.0569 rpy=0 0 0, axis 0 0 1, limit lower=-6.2831853 upper=6.2831853 effort=370 velocity=1.4363
- added joint joint_arm2: type revolute, parent link_arm1, child link_arm2, origin xyz=0 0 0.1931 rpy=0 0 0, axis 0 1 0, limit lower=-2.0943951 upper=2.0943951 effort=370 velocity=1.4363
- added joint joint_arm3: type revolute, parent link_arm2, child link_arm3, origin xyz=0 0 0.110 rpy=0 0 0, axis 0 0 1, limit lower=-6.2831853 upper=6.2831853 effort=176 velocity=1.4189
- added joint joint_arm4: type revolute, parent link_arm3, child link_arm4, origin xyz=0 0 0.298 rpy=0 0 0, axis 0 1 0, limit lower=-2.0943951 upper=2.0943951 effort=176 velocity=1.4189
- added joint joint_arm5: type revolute, parent link_arm4, child link_arm5, origin xyz=0 0 0.100 rpy=0 0 0, axis 0 0 1, limit lower=-6.2831853 upper=6.2831853 effort=41.6 velocity=1.4363
- added joint joint_arm6: type revolute, parent link_arm5, child link_arm6, origin xyz=0 0 0.2165 rpy=0 0 0, axis 0 1 0, limit lower=-2.0943951 upper=2.0943951 effort=20.1 velocity=1.4363
- added joint joint_arm7: type revolute, parent link_arm6, child link_arm7, origin xyz=0 0 0.080 rpy=0 0 0, axis 0 0 1, limit lower=-6.2831853 upper=6.2831853 effort=9.6 velocity=1.8727

Commit message: improved arm controller

File: cob3_simulation/cob3_defs/ros/defs/arm.urdf (robot description, URDF)
Before this commit: robot arm, 8 links, 7 joints
Joints:
- joint joint_arm1: limit lower=-6.2831853 upper=6.2831853 effort=370 velocity=1.4363 -> lower=-6.2831853 upper=6.2831853 effort=370 velocity=0.4363
- joint joint_arm2: limit lower=-2.0943951 upper=2.0943951 effort=370 velocity=1.4363 -> lower=-2.0943951 upper=2.0943951 effort=370 velocity=0.4363
- joint joint_arm3: limit lower=-6.2831853 upper=6.2831853 effort=176 velocity=1.4189 -> lower=-6.2831853 upper=6.2831853 effort=176 velocity=0.4189
- joint joint_arm4: limit lower=-2.0943951 upper=2.0943951 effort=176 velocity=1.4189 -> lower=-2.0943951 upper=2.0943951 effort=176 velocity=0.4189
- joint joint_arm5: limit lower=-6.2831853 upper=6.2831853 effort=41.6 velocity=1.4363 -> lower=-6.2831853 upper=6.2831853 effort=41.6 velocity=0.4363
- joint joint_arm6: limit lower=-2.0943951 upper=2.0943951 effort=20.1 velocity=1.4363 -> lower=-2.0943951 upper=2.0943951 effort=20.1 velocity=0.4363
- joint joint_arm7: limit lower=-6.2831853 upper=6.2831853 effort=9.6 velocity=1.8727 -> lower=-6.2831853 upper=6.2831853 effort=9.6 velocity=0.8727
