Commit message: added head_cover

File: cob3_simulation/cob3_defs/ros/defs/torso.urdf (robot description, URDF)
Before this commit: robot torso, 18 links, 17 joints
Links:
- added link link_head_cover, mass 1; collision mesh filename=package://cob3_defs/common/files/meshes/head_cover.stl; visual mesh filename=package://cob3_defs/common/files/meshes/head_cover.stl
- link link_tray: geometry collision mesh filename=package://cob3_defs/common/files/meshes/tray.stl; visual mesh filename=package://cob3_defs/common/files/meshes/tray.stl
Joints:
- added joint joint_headZ_head_cover: type fixed, parent link_head, child link_head_cover, origin xyz=0 0 0 rpy=0 0 0
- joint joint_platform_tray: axis 0 0 1 -> 0 1 1; limit lower=-1 upper=1 effort=100 velocity=5 -> lower=-2 upper=3 effort=100 velocity=5; origin xyz=0.5 0 0.8 rpy=0 0 0 -> xyz=0.21864 0.20061 0.83196 rpy=0 0 0

File: cob3_simulation/cob3_defs/ros/robots/cob3.urdf.xacro (robot description, xacro)
@@ -19,5 +19,5 @@
 	<include filename="$(find cob3_defs)/ros/defs/arm.urdf" />
 	<joint name="joint_platform_arm0" type="fixed">
-		<origin xyz="0 0 0.8" rpy="0.5 0 0" /> <!-- TODO: put in real transformation from platform to arm0-->
+		<origin xyz="0 0 0.8" rpy="0.5 0 -0.5" /> <!-- TODO: put in real transformation from platform to arm0-->
 		<parent link="link_platform"/>
 		<child link="link_arm0"/>

Commit message: update of torso description

File: cob3_simulation/cob3_defs/ros/defs/torso.urdf (robot description, URDF)
Before this commit: robot torso, 19 links, 18 joints
Joints:
- joint joint_platform_tray: axis 0 1 1 -> 0 0 1; limit lower=-2 upper=3 effort=100 velocity=5 -> lower=0 upper=3.31612 effort=100 velocity=5; origin xyz=0.21864 0.20061 0.83196 rpy=0 0 0 -> xyz=0.21864 0.20061 0.83196 rpy=-0.707 0 0

Commit message: lifted tray

File: cob3_simulation/cob3_defs/ros/defs/torso.urdf (robot description, URDF)
Before this commit: robot torso, 19 links, 18 joints
Joints:
- joint joint_platform_tray: origin xyz=0.21864 0.20061 0.83196 rpy=-0.707 0 0 -> xyz=0.21864 0.20061 0.73196 rpy=-0.707 0 0
