Commit message: configure sdh controller and setup

File: cob3_simulation/cob3_defs/ros/robots/cob3_sdh.urdf.xacro (robot description, xacro)
@@ -7,18 +7,18 @@
 	<link name="link_arm7">
 		<inertial>
-			<origin xyz="0 0 0.05625" rpy="0 0 0"/>
-			<mass value="1000"/>
-			<inertia ixx="1000"  ixy="0"  ixz="0" iyy="1000" iyz="0" izz="1000" />
+			<origin xyz="0 0 0" rpy="0 0 0"/>
+			<mass value="2000"/>
+			<inertia ixx="1"  ixy="0"  ixz="0" iyy="1" iyz="0" izz="1" />
 		</inertial>
 		<visual>
-			<origin xyz="0 0 0.05625" rpy="0 0 0" />
+			<origin xyz="0 0 0" rpy="0 0 0" />
 			<geometry>
-				<cylinder radius="0.1" length="0.1125"/>
+				<mesh filename="package://cob3_defs/common/files/meshes/arm7.stl" />
 			</geometry>
 		</visual>
 		<collision>
-			<origin xyz="0 0 0.05625" rpy="0 0 0" />
+			<origin xyz="0 0 0" rpy="0 0 0" />
 			<geometry>
-				<cylinder radius="0.1" length="0.1125"/> <!-- TODO put in real offset of arm7 -->
+				<mesh filename="package://cob3_defs/common/files/meshes/arm7.stl"/>
 			</geometry>
 		</collision>

Commit message: adjust armTCP offset

File: cob3_simulation/cob3_defs/ros/robots/cob3_sdh.urdf.xacro (robot description, xacro)
@@ -12,13 +12,15 @@
 		</inertial>
 		<visual>
-			<origin xyz="0 0 0" rpy="0 0 0" />
+			<origin xyz="0 0 0.0563" rpy="0 0 0" />
 			<geometry>
-				<mesh filename="package://cob3_defs/common/files/meshes/arm7.stl" />
+		        <box size="0.1 0.1 0.1126"/>
+<!--				<mesh filename="package://cob3_defs/common/files/meshes/arm7.stl" /> -->
 			</geometry>
 		</visual>
 		<collision>
-			<origin xyz="0 0 0" rpy="0 0 0" />
+			<origin xyz="0 0 0.0563" rpy="0 0 0" />
 			<geometry>
-				<mesh filename="package://cob3_defs/common/files/meshes/arm7.stl"/>
+		        <box size="0.1 0.1 0.1126"/>
+<!--				<mesh filename="package://cob3_defs/common/files/meshes/arm7.stl"/> -->
 			</geometry>
 		</collision>
