Commit message: added platform and modifications to torso, arm and sdh

File: cob3_simulation/cob3_defs/ros/robots/cob3_torso.urdf (robot description, URDF)
Before this commit: robot cob3_torso, 10 links, 10 joints
Joints:
- joint joint_world_torso: origin xyz=0 0 0.1126 rpy=0 0 0 -> xyz=0 0 0 rpy=0 0 0

File: cob3_simulation/cob3_defs/ros/robots/cob3_torso_arm_sdh.urdf.xacro (robot description, xacro)
@@ -6,11 +6,15 @@
 	<!-- include gazebo defs-->
 	<include filename="$(find cob3_defs)/ros/defs/gazebo.urdf" />
-	<!-- include torso defs-->
-	<include filename="$(find cob3_defs)/ros/defs/platform.urdf" />
+	<!-- create joint to world -->
+	<joint name="joint_world_torso" type="fixed">
+		<origin xyz="0 0 0" rpy="0 0 0" />
+		<parent link="world"/>
+		<child link="link_torso"/>
+	</joint>
 	<!-- include torso defs-->
 	<include filename="$(find cob3_defs)/ros/defs/torso.urdf" />
 	<joint name="joint_basePlate_torso" type="fixed">
-		<origin xyz="0 0 0.5" rpy="0 0 0" />
-		<parent link="link_platform"/>
+		<origin xyz="0 0 0.1126" rpy="0 0 0" />
+		<parent link="link_base_Plate"/>
 		<child link="link_torso"/>
 	</joint>
